File: kicad/Dolly driver.kicad_pcb (KiCad board)
At the start: 2 copper layers, 43 x 43 mm, 11 parts, among them J1 Barrel_Jack_MountingPin, M1 Stepper_Motor_bipolar, SW1 SW_Push, SW2 SW_Push, U1 ProMicro, U2 AMS1117-5.0

Commit message: fix(kicad): correct net numbering and update pad connections in Dolly driver PCB
- Renumber nets for consistency and correct sequencing
- Update pad net assignments to reflect new net numbers
- Adjust thermal bridge width and gap for enable pad
- Remove redundant pinfunction and pintype entries
- Ensure GND and VMOT net references are aligned correctly
- Correct pinfunction and pintype assignments for clarity
- Remove unconnected net labels and rename to proper nets where applicable
- Fix net indices in segment and drill definitions for accuracy
Connections:
- A1 pad 9: unconnected-(A1-~{ENABLE}-Pad9) -> GND
