File: kicad/Dolly driver.kicad_sch (KiCad schematic)
At the start: 11 parts, among them J1 Barrel_Jack_MountingPin, M1 Stepper_Motor_bipolar, SW1 SW_Push, SW2 SW_Push, U1 ProMicro, U2 AMS1117-5.0

Commit message: fix(kicad): correct net numbering and update pad connections in Dolly driver PCB
- Renumber nets for consistency and correct sequencing
- Update pad net assignments to reflect new net numbers
- Adjust thermal bridge width and gap for enable pad
- Remove redundant pinfunction and pintype entries
- Ensure GND and VMOT net references are aligned correctly
- Correct pinfunction and pintype assignments for clarity
- Remove unconnected net labels and rename to proper nets where applicable
- Fix net indices in segment and drill definitions for accuracy
Connections:
- net GND: now also A1.9 (~{ENABLE})
Changed lines of the file:
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@@
+	)
+	(symbol
+		(lib_id "power:GND")
+		(at 196.85 127 270)
+		(unit 1)
+		(exclude_from_sim no)
+		(in_bom yes)
+		(on_board yes)
+		(dnp no)
+		(fields_autoplaced yes)
+		(property "Reference" "#PWR04"
+			(at 190.5 127 0)
+			(effects
+				(font
+					(size 1.27 1.27)
+				)
+				(hide yes)
+			)
+		)
+		(property "Value" "GND"
+			(at 193.6751 127 90)
+			(effects
+				(font
+					(size 1.27 1.27)
+				)
+				(justify right)
+			)
+		)
+		(property "Footprint" ""
+			(at 196.85 127 0)
+			(effects
+				(font
+					(size 1.27 1.27)
+				)
+				(hide yes)
+			)
+		)
+		(property "Datasheet" ""
+			(at 196.85 127 0)
+			(effects
+				(font
+					(size 1.27 1.27)
+				)
+				(hide yes)
+			)
+		)
+		(property "Description" "Power symbol creates a global label with name \"GND\" , ground"
+			(at 196.85 127 0)
+			(effects
+				(font
+					(size 1.27 1.27)
+				)
+				(hide yes)
+			)
+		)
+		(pin "1"
+		)
+		(instances
+			(project ""
+				(path "/dd698658-9777-4277-b999-ca021351db53"
+					(reference "#PWR04")
+					(unit 1)
+				)
+			)
+		)
 	)
 	(symbol
